Commit message: lacquey gripper working

File: automatica2014_description/urdf/ur5.urdf.xacro (robot description, xacro)
@@ -13,8 +13,8 @@
     <joint name="gripper_joint" type="fixed" >
         <parent link="ur5_wrist_3_link" />
-        <child link="gripper_grasp_link" />
+        <child link="gripper_link" />
         <origin xyz="0.0 0.06 0.0" rpy="1.57 0 0"/>
     </joint>
-    <link name="gripper_grasp_link">
+    <link name="gripper_link">
         <visual>
             <geometry>
@@ -29,10 +29,10 @@
     </link>
      <joint name="finger_left_joint" type="continuous" >
-        <parent link="gripper_grasp_link" />
+        <parent link="gripper_link" />
         <child link="finger_left_link" />
         <limit effort="100" lower="-0.01" upper="0.062" velocity="1.0"/>
         <calibration rising="0.0"/>
         <origin xyz="-0.03 -0.03 -0.07" rpy="-1.57 0 0"/>
-        <axis xyz="0 0 1" />
+        <axis xyz="-1 0 0" />
     </joint>
     <link name="finger_left_link">
@@ -55,10 +55,10 @@
     </link>
      <joint name="finger_right_joint" type="continuous" >
-        <parent link="gripper_grasp_link" />
+        <parent link="gripper_link" />
         <child link="finger_right_link" />
         <limit effort="100" lower="-0.01" upper="0.062" velocity="1.0"/>
         <calibration rising="0.0"/>
         <origin xyz="0.0 0.03 -0.07" rpy="-1.57 0 3.14"/>
-        <axis xyz="0 0 1" />
+        <axis xyz="-1 0 0" />
     </joint>
     <link name="finger_right_link">
@@ -80,3 +80,9 @@
         </collision>
     </link>
+    <joint name="gripper_grasp_joint" type="fixed" >
+        <parent link="gripper_link" />
+        <child link="gripper_grasp_link" />
+        <origin xyz="0.0 0.06 0.0" rpy="1.57 0 0"/>
+    </joint>
+    <link name="gripper_grasp_link"/>
 </robot>

Commit message: fix ur5 gripper links

File: automatica2014_description/urdf/ur5.urdf.xacro (robot description, xacro)
@@ -12,7 +12,7 @@
     <!-- gripper -->
     <joint name="gripper_joint" type="fixed" >
-        <parent link="ur5_wrist_3_link" />
+        <parent link="ur5_ee_link" />
         <child link="gripper_link" />
-        <origin xyz="0.0 0.06 0.0" rpy="1.57 0 0"/>
+        <origin xyz="0.0 0.0 0.0" rpy="1.57 3.14 -1.57"/>
     </joint>
     <link name="gripper_link">
@@ -83,5 +83,5 @@
         <parent link="gripper_link" />
         <child link="gripper_grasp_link" />
-        <origin xyz="0.0 0.06 0.0" rpy="3.14 0 -1.5708"/>
+        <origin xyz="0.0 0.0 -0.12" rpy="0 0 1.57"/>
     </joint>
     <link name="gripper_grasp_link"/>

Commit message: move gripper_grasp_link for ur5

File: automatica2014_description/urdf/ur5.urdf.xacro (robot description, xacro)
@@ -83,5 +83,5 @@
         <parent link="gripper_link" />
         <child link="gripper_grasp_link" />
-        <origin xyz="0.0 0.0 -0.12" rpy="0 0 1.57"/>
+        <origin xyz="0.0 0.0 -0.18" rpy="0 0 1.57"/>
     </joint>
     <link name="gripper_grasp_link"/>

Commit message: fix limits of gripper

File: automatica2014_description/urdf/ur5.urdf.xacro (robot description, xacro)
@@ -31,5 +31,5 @@
         <parent link="gripper_link" />
         <child link="finger_left_link" />
-        <limit effort="100" lower="-0.01" upper="0.062" velocity="1.0"/>
+        <limit effort="100" lower="-0.01" upper="2" velocity="1.0"/>
         <calibration rising="0.0"/>
         <origin xyz="-0.03 -0.03 -0.07" rpy="-1.57 0 0"/>
@@ -57,5 +57,5 @@
         <parent link="gripper_link" />
         <child link="finger_right_link" />
-        <limit effort="100" lower="-0.01" upper="0.062" velocity="1.0"/>
+        <limit effort="100" lower="-0.01" upper="2" velocity="1.0"/>
         <calibration rising="0.0"/>
         <origin xyz="0.0 0.03 -0.07" rpy="-1.57 0 3.14"/>

Commit message: add collision to gripper grasp link of lacquey

File: automatica2014_description/urdf/ur5.urdf.xacro (robot description, xacro)
@@ -85,4 +85,11 @@
         <origin xyz="0.0 0.0 -0.18" rpy="0 0 1.57"/>
     </joint>
-    <link name="gripper_grasp_link"/>
+    <link name="gripper_grasp_link" >
+        <collision>
+            <origin xyz="0.0 0.0 0.15" rpy="0 0 0"/>
+            <geometry>
+                <box size="0.01 0.01 0.01"/>
+            </geometry>
+        </collision>
+    </link>
 </robot>

Commit message: updated lacquey gripper

File: automatica2014_description/urdf/ur5.urdf.xacro (robot description, xacro)
@@ -1,4 +1,5 @@
 <robot xmlns:xacro="http://ros.org/wiki/xacro" name="ur5">
     <xacro:include filename="$(find ur_description)/urdf/ur5_joint_limited.urdf.xacro" />
+    <xacro:include filename="$(find automatica2014_description)/urdf/lacquey.urdf.xacro" />
     <!-- cell -->
     <xacro:include filename="$(find automatica2014_description)/urdf/cell.urdf.xacro" />
@@ -10,78 +11,12 @@
     </joint>
     <xacro:ur5_robot prefix="ur5_"/>
+    <xacro:lacquey_gripper prefix="" parent="ur5_ee_link">
+        <origin xyz="0.0 0.0 0.0" rpy="0 1.57 0"/>
+    </xacro:lacquey_gripper>
     <!-- gripper -->
-    <joint name="gripper_joint" type="fixed" >
-        <parent link="ur5_ee_link" />
-        <child link="gripper_link" />
-        <origin xyz="0.0 0.0 0.0" rpy="1.57 3.14 -1.57"/>
-    </joint>
-    <link name="gripper_link">
-        <visual>
-            <geometry>
-                <mesh filename="package://automatica2014_description/meshes/gripper_base_lacquey.stl"/>
-            </geometry>
-        </visual>
-        <collision>
-            <geometry>
-                <mesh filename="package://automatica2014_description/meshes/gripper_base_lacquey.stl"/>
-            </geometry>
-        </collision>
-    </link>
-     <joint name="finger_left_joint" type="continuous" >
-        <parent link="gripper_link" />
-        <child link="finger_left_link" />
-        <limit effort="100" lower="-0.01" upper="2" velocity="1.0"/>
-        <calibration rising="0.0"/>
-        <origin xyz="-0.03 -0.03 -0.07" rpy="-1.57 0 0"/>
-        <axis xyz="-1 0 0" />
-    </joint>
-    <link name="finger_left_link">
-        <visual>
-            <geometry>
-                <mesh filename="package://automatica2014_description/meshes/finger_right_lacquey.stl"/>
-            </geometry>
-            <material name="blue">
-                <color rgba="0 0 1 1"/>
-            </material>
-        </visual>
-        <collision>
-            <geometry>
-                <mesh filename="package://automatica2014_description/meshes/finger_right_lacquey.stl"/>
-            </geometry>
-            <material name="blue">
-                <color rgba="0 0 1 1"/>
-            </material>
-        </collision>
-    </link>
-     <joint name="finger_right_joint" type="continuous" >
-        <parent link="gripper_link" />
-        <child link="finger_right_link" />
-        <limit effort="100" lower="-0.01" upper="2" velocity="1.0"/>
-        <calibration rising="0.0"/>
-        <origin xyz="0.0 0.03 -0.07" rpy="-1.57 0 3.14"/>
-        <axis xyz="-1 0 0" />
-    </joint>
-    <link name="finger_right_link">
-        <visual>
-            <geometry>
-                <mesh filename="package://automatica2014_description/meshes/finger_left_lacquey.stl"/>
-            </geometry>
-            <material name="blue">
-                <color rgba="0 0 1 1"/>
-            </material>
-        </visual>
-        <collision>
-            <geometry>
-                <mesh filename="package://automatica2014_description/meshes/finger_left_lacquey.stl"/>
-            </geometry>
-                <material name="blue">
-                <color rgba="0 0 1 1"/>
-            </material>
-        </collision>
-    </link>
     <joint name="gripper_grasp_joint" type="fixed" >
         <parent link="gripper_link" />
         <child link="gripper_grasp_link" />
-        <origin xyz="0.0 0.0 -0.18" rpy="0 0 1.57"/>
+        <origin xyz="0.0 0.0 0.18" rpy="3.14 0 0"/>
     </joint>
     <link name="gripper_grasp_link" >
