Commit message: brin gcamera in positoin

File: automatica2014_description/urdf/cell.urdf.xacro (robot description, xacro)
@@ -1,5 +1,5 @@
 <robot xmlns:xacro="http://ros.org/wiki/xacro">
     <xacro:property name="cam3d_env_origin">
-        <origin xyz="0 0 0" rpy="0 0 0" />
+        <origin xyz="1 1 2" rpy="3.14 0 0" />
     </xacro:property>
     <xacro:property name="cam3d_mon_origin">

Commit message: add camera calibration link

File: automatica2014_description/urdf/cell.urdf.xacro (robot description, xacro)
@@ -3,5 +3,5 @@
         <origin xyz="0 0 0" rpy="0 0 0" />
     </xacro:property>
-    <xacro:property name="cam3d_mon_origin">
+    <xacro:property name="cam3d_calibration_origin">
         <origin xyz="0 0 0" rpy="0 0 0" />
     </xacro:property>

File: automatica2014_description/urdf/workspace.urdf.xacro (robot description, xacro)
@@ -8,7 +8,10 @@
         <xacro:insert_block name="cam3d_env_origin" />
     </xacro:cob_kinect_v0>
-    <!-- monitor camera -->
-    <xacro:cob_kinect_v0 name="cam3d_mon" ros_topic="cam3d_mon" parent="base_link">
-        <xacro:insert_block name="cam3d_mon_origin" />
-    </xacro:cob_kinect_v0>
+    <!-- camera calibration link -->
+    <link name="cam3d_calibration_link"/>
+    <joint name="camera_calibration_joint" type="fixed" >
+        <parent link="base_link" />
+        <child link="cam3d_calibration_link" />
+        <xacro:insert_block name="cam3d_calibration_origin" />
+    </joint>
 </robot>

Commit message: rough calibration without clipping

File: automatica2014_description/urdf/cell.urdf.xacro (robot description, xacro)
@@ -1,5 +1,5 @@
 <robot xmlns:xacro="http://ros.org/wiki/xacro">
     <xacro:property name="cam3d_env_origin">
-        <origin xyz="1 1 2" rpy="3.14 0 0" />
+        <origin xyz="0.6 1.1 1.65" rpy="3.14 0 0" />
     </xacro:property>
     <xacro:property name="cam3d_calibration_origin">

Commit message: fix camera position and visualization

File: automatica2014_description/urdf/cell.urdf.xacro (robot description, xacro)
@@ -1,5 +1,5 @@
 <robot xmlns:xacro="http://ros.org/wiki/xacro">
     <xacro:property name="cam3d_env_origin">
-        <origin xyz="0.6 1.1 1.65" rpy="3.14 0 0" />
+        <origin xyz="0.6 1.1 1.65" rpy="3.14 0 3.14" />
     </xacro:property>
     <xacro:property name="cam3d_calibration_origin">

Commit message: calibration done

File: automatica2014_description/urdf/cell.urdf.xacro (robot description, xacro)
@@ -1,19 +1,19 @@
 <robot xmlns:xacro="http://ros.org/wiki/xacro">
-    <xacro:property name="cam3d_env_origin">
-        <origin xyz="0.6 1.1 1.65" rpy="3.14 0 3.14" />
+    <xacro:property name="cam3d_calibration_origin">
+        <origin xyz="0.65 0.791 0" rpy="0 0 0" />
     </xacro:property>
-    <xacro:property name="cam3d_calibration_origin">
-        <origin xyz="0 0 0" rpy="0 0 0" />
+    <xacro:property name="cam3d_env_origin"> <!-- fill in calibration values here -->
+        <origin xyz="-0.00525894500153 0.263612777206 1.7" rpy="-3.1415926 0 -3.1415926" />
     </xacro:property>
     <xacro:property name="ur5_origin">
-        <origin xyz="0.5 1.5 0" rpy="0 0 0" />
+        <origin xyz="0.45 1.585 0.01" rpy="0 0 0" />
     </xacro:property>
     <xacro:property name="sia10f_origin">
-        <origin xyz="0.5 0.5 0" rpy="0 0 0" />
+        <origin xyz="0.45 0.35 0.015" rpy="0 0 0" />
     </xacro:property>
     <link name="base_link">
         <visual>
             <geometry>
-            <mesh filename="package://automatica2014_description/meshes/cell.stl" scale="0.001 0.001 0.001"/>
+                <mesh filename="package://automatica2014_description/meshes/cell.stl" scale="0.001 0.001 0.001"/>
             </geometry>
         </visual>

File: automatica2014_description/urdf/workspace.urdf.xacro (robot description, xacro)
@@ -5,12 +5,12 @@
     <xacro:include filename="$(find automatica2014_description)/urdf/cell.urdf.xacro" />
     <!-- environment camera -->
-    <xacro:cob_kinect_v0 name="cam3d_env" ros_topic="cam3d_env" parent="base_link">
+    <xacro:cob_kinect_v0 name="cam3d_env" ros_topic="cam3d_env" parent="cam3d_calibration_link">
         <xacro:insert_block name="cam3d_env_origin" />
     </xacro:cob_kinect_v0>
     <!-- camera calibration link -->
-    <link name="marker"/>
-    <joint name="camera_calibration_joint" type="fixed" >
+    <link name="cam3d_calibration_link"/>
+    <joint name="cam3d_calibration_joint" type="fixed" >
         <parent link="base_link" />
-        <child link="marker" />
+        <child link="cam3d_calibration_link" />
         <xacro:insert_block name="cam3d_calibration_origin" />
     </joint>

Commit message: gripper grasp link

File: automatica2014_description/urdf/cell.urdf.xacro (robot description, xacro)
@@ -7,5 +7,5 @@
     </xacro:property>
     <xacro:property name="ur5_origin">
-        <origin xyz="0.45 1.585 0.01" rpy="0 0 0" />
+        <origin xyz="0.45 1.585 0.01" rpy="0 0 -0.7854" />
     </xacro:property>
     <xacro:property name="sia10f_origin">

File: automatica2014_description/urdf/sia10f.urdf.xacro (robot description, xacro)
@@ -45,5 +45,5 @@
                     <parent link="gripper_link" />
                     <child link="gripper_grasp_link" />
-                    <origin xyz="0.0 0.0 0.0" rpy="0 0 0"/>
+                    <origin xyz="0.0 0.0 0.12" rpy="0 3.14 1.5708"/>
                 </joint>
                 <link name="gripper_grasp_link" />

Commit message: add base_footprint

File: automatica2014_description/urdf/cell.urdf.xacro (robot description, xacro)
@@ -1,3 +1,6 @@
 <robot xmlns:xacro="http://ros.org/wiki/xacro">
+    <xacro:property name="base_origin">
+        <origin xyz="0 0 1.0" rpy="0 0 0" />
+    </xacro:property>
     <xacro:property name="cam3d_calibration_origin">
         <origin xyz="0.65 0.791 0" rpy="0 0 0" />
@@ -12,4 +15,10 @@
         <origin xyz="0.45 0.35 0.015" rpy="0 0 0" />
     </xacro:property>
+    <link name="base_footprint"/>
+    <joint name="base_joint" type="fixed" >
+        <parent link="base_footprint" />
+        <child link="base_link" />
+        <xacro:insert_block name="base_origin" />
+    </joint>
     <link name="base_link">
         <visual>

Commit message: fix calibration

File: automatica2014_description/urdf/cell.urdf.xacro (robot description, xacro)
@@ -1,5 +1,5 @@
 <robot xmlns:xacro="http://ros.org/wiki/xacro">
     <xacro:property name="base_origin">
-        <origin xyz="0 0 1.0" rpy="0 0 0" />
+        <origin xyz="0 0 0.95" rpy="0 0 0" />
     </xacro:property>
     <xacro:property name="cam3d_calibration_origin">
@@ -7,11 +7,13 @@
     </xacro:property>
     <xacro:property name="cam3d_env_origin"> <!-- fill in calibration values here -->
-        <origin xyz="-0.00525894500153 0.263612777206 1.7" rpy="-3.1415926 0 -3.1415926" />
+        <origin xyz="-0.00525894500153 0.263612777206 1.65" rpy="-3.1415926 0 -3.1415926" />
     </xacro:property>
     <xacro:property name="ur5_origin">
-        <origin xyz="0.45 1.585 0.01" rpy="0 0 -0.7854" />
+        <!--origin xyz="0.45 1.585 0.01" rpy="0 0 -0.7854" /--> <!-- measured -->
+        <origin xyz="0.45 1.55 0.01" rpy="0 0 -0.7854" /> <!-- manually calibrated -->
     </xacro:property>
     <xacro:property name="sia10f_origin">
-        <origin xyz="0.45 0.35 0.015" rpy="0 0 0" />
+        <!--origin xyz="0.45 0.35 0.015" rpy="0 0 0" /--> <!-- measured -->
+        <origin xyz="0.45 0.37 0.015" rpy="0 0 0" /> <!-- manually calibrated -->
     </xacro:property>
     <link name="base_footprint"/>

Commit message: turned ur5

File: automatica2014_description/urdf/cell.urdf.xacro (robot description, xacro)
@@ -11,5 +11,5 @@
     <xacro:property name="ur5_origin">
         <!--origin xyz="0.45 1.585 0.01" rpy="0 0 -0.7854" /--> <!-- measured -->
-        <origin xyz="0.45 1.55 0.01" rpy="0 0 -0.7854" /> <!-- manually calibrated -->
+        <origin xyz="0.45 1.55 0.01" rpy="0 0 -2.35619449019" /> <!-- manually calibrated -->
     </xacro:property>
     <xacro:property name="sia10f_origin">

Commit message: new calibration

File: automatica2014_description/urdf/cell.urdf.xacro (robot description, xacro)
@@ -1,2 +1,3 @@
+<?xml version="1.0"?>
 <robot xmlns:xacro="http://ros.org/wiki/xacro">
     <xacro:property name="base_origin">
@@ -7,13 +8,14 @@
     </xacro:property>
     <xacro:property name="cam3d_env_origin"> <!-- fill in calibration values here -->
-        <origin xyz="-0.00525894500153 0.263612777206 1.65" rpy="-3.1415926 0 -3.1415926" />
+        <!--origin xyz="-0.00525894500153 0.263612777206 1.65" rpy="-3.1415926 0 -3.1415926" /-->
+        <origin xyz="-0.00549884192955 0.273024997864 1.80" rpy="-3.1415926 0 -3.1415926" />
     </xacro:property>
     <xacro:property name="ur5_origin">
-        <!--origin xyz="0.45 1.585 0.01" rpy="0 0 -0.7854" /--> <!-- measured -->
-        <origin xyz="0.45 1.55 0.01" rpy="0 0 -2.35619449019" /> <!-- manually calibrated -->
+        <origin xyz="0.45 1.585 0.01" rpy="0 0 -2.35619449019" /> <!-- measured -->
+        <!--origin xyz="0.45 1.55 0.01" rpy="0 0 -2.35619449019" /--> <!-- manually calibrated -->
     </xacro:property>
     <xacro:property name="sia10f_origin">
-        <!--origin xyz="0.45 0.35 0.015" rpy="0 0 0" /--> <!-- measured -->
-        <origin xyz="0.45 0.37 0.015" rpy="0 0 0" /> <!-- manually calibrated -->
+        <origin xyz="0.45 0.35 0.015" rpy="0 0 0" /> <!-- measured -->
+        <!--origin xyz="0.45 0.37 0.015" rpy="0 0 0" /--> <!-- manually calibrated -->
     </xacro:property>
     <link name="base_footprint"/>

Commit message: fix sia10f settings

File: automatica2014_description/urdf/cell.urdf.xacro (robot description, xacro)
@@ -16,5 +16,5 @@
     </xacro:property>
     <xacro:property name="sia10f_origin">
-        <origin xyz="0.45 0.35 0.015" rpy="0 0 0" /> <!-- measured -->
+        <origin xyz="0.605 0.553 0.015" rpy="0 0 1.5708" /> <!-- measured -->
         <!--origin xyz="0.45 0.37 0.015" rpy="0 0 0" /--> <!-- manually calibrated -->
     </xacro:property>

File: automatica2014_description/urdf/gripper.urdf.xacro (robot description, xacro)
@@ -57,5 +57,5 @@
         <parent link="gripper_link" />
         <child link="finger_left_link" />
-        <limit effort="100" lower="-0.01" upper="0.062" velocity="1.0"/>
+        <limit effort="100" lower="0.001" upper="0.031" velocity="2.0"/>
         <calibration rising="0.0"/>
         <origin xyz="0.0 -0.008 0.096" rpy="-1.57 -1.57 3.14"/>
@@ -65,5 +65,5 @@
             <parent link="gripper_link" />
             <child link="finger_right_link" />
-            <limit effort="100" lower="-0.01" upper="0.062" velocity="1.0"/>
+            <limit effort="100" lower="0.001" upper="0.031" velocity="2.0"/>
             <calibration rising="0.0"/>
             <origin xyz="0.0 0.008 0.096" rpy="-1.57 -1.57 0"/>

File: automatica2014_description/urdf/sia10f.urdf.xacro (robot description, xacro)
@@ -1,5 +1,5 @@
     <robot xmlns:xacro="http://ros.org/wiki/xacro" name="sia10f">
                 <xacro:property name="gripper_origin">
-                    <origin xyz="0. 0. 0" rpy="0 0 0" />
+                    <origin xyz="0. 0. 0.0225" rpy="0 0 0" />
                 </xacro:property>
                 <xacro:property name="flange_origin">
@@ -45,5 +45,5 @@
                     <parent link="gripper_link" />
                     <child link="gripper_grasp_link" />
-                    <origin xyz="0.0 0.0 0.12" rpy="0 3.14 1.5708"/>
+                    <origin xyz="0.0 0.0 0.14" rpy="0 3.14 1.5708"/>
                 </joint>
                 <link name="gripper_grasp_link" />

Commit message: new cell mesh

File: automatica2014_description/urdf/cell.urdf.xacro (robot description, xacro)
@@ -1,4 +1,4 @@
 <?xml version="1.0"?>
-<robot xmlns:xacro="http://ros.org/wiki/xacro">
+<robot xmlns:xacro="http://ros.org/wiki/xacro" name="cell">
     <xacro:property name="base_origin">
         <origin xyz="0 0 0.95" rpy="0 0 0" />
@@ -28,5 +28,5 @@
         <visual>
             <geometry>
-                <mesh filename="package://automatica2014_description/meshes/cell.stl" scale="0.001 0.001 0.001"/>
+                <mesh filename="package://automatica2014_description/meshes/cell.dae" scale="1 1 1"/>
             </geometry>
         </visual>
