Commit message: URDF modifications to contain the fingers

File: automatica2014_description/urdf/gripper.urdf.xacro (robot description, xacro)
@@ -6,4 +6,40 @@
         <origin xyz="0. 0. 0.03" rpy="0. 0 0" />
     </xacro:property>
+     <link name="finger_left_link">
+        <visual>
+            <geometry>
+            <mesh filename="package://automatica2014_description/meshes/finger_left.stl"/>
+            </geometry>
+            <material name="silver">
+					<color rgba="1 1 1 1"/>
+			</material>
+        </visual>
+        <collision>
+            <geometry>
+                <mesh filename="package://automatica2014_description/meshes/finger_left.stl"/>
+            </geometry>
+            <material name="silver">
+					<color rgba="1 1 1 1"/>
+			</material>
+        </collision>
+    </link>
+    <link name="finger_right_link">
+        <visual>
+            <geometry>
+            <mesh filename="package://automatica2014_description/meshes/finger_right.stl"/>
+            </geometry>
+            <material name="silver">
+					<color rgba="1 1 1 1"/>
+			</material>
+        </visual>
+        <collision>
+            <geometry>
+                <mesh filename="package://automatica2014_description/meshes/finger_right.stl"/>
+            </geometry>
+            <material name="silver">
+					<color rgba="1 1 1 1"/>
+			</material>
+        </collision>
+    </link>
     <link name="gripper_grasp_link">
         <visual>
@@ -11,6 +47,6 @@
             <mesh filename="package://automatica2014_description/meshes/gripper.stl" scale="0.001 0.001 0.001"/>
             </geometry>
-            <material name="silver">
-					<color rgba="0.8 0.8 0.8 1"/>
+            <material name="blue">
+					<color rgba="0 0 1 1"/>
 			</material>
         </visual>
@@ -19,6 +55,6 @@
                 <mesh filename="package://automatica2014_description/meshes/gripper.stl" scale="0.001 0.001 0.001"/>
             </geometry>
-            <material name="silver">
-					<color rgba="0.8 0.8 0.8 1"/>
+            <material name="blue">
+					<color rgba="0 0 1 1"/>
 			</material>
         </collision>

File: automatica2014_description/urdf/sia10f.urdf.xacro (robot description, xacro)
@@ -1,4 +1,3 @@
-	<?xml version="1.0"?>
-	<robot xmlns:xacro="http://ros.org/wiki/xacro" name="sia10f">
+    <robot xmlns:xacro="http://ros.org/wiki/xacro" name="sia10f">
 		<xacro:include filename="$(find motoman_sia10f_support)/urdf/sia10f_macro.xacro" />
 		<!-- cell -->
@@ -23,6 +22,21 @@
 		    <parent link="gripper_flange_link" />
 		    <child link="gripper_grasp_link" />
+		    <xacro:insert_block name="gripper_origin" />
+		</joint>
+		<joint name="finger_left_joint" type="fixed" >
+		    <parent link="gripper_grasp_link" />
+		    <child link="finger_left_link" />
+		    <limit effort="100" lower="-0.1" upper="1.1" velocity="1.0"/>
+		    <calibration rising="0.0"/>
+		    <origin xyz="0.0 0.044 0.076" rpy="-1.57 0 0"/>
+		    <axis xyz="0 0 0" />
+		</joint>
+		<joint name="finger_right_joint" type="fixed" >
+		    <parent link="gripper_grasp_link" />
+		    <child link="finger_right_link" />
 		<limit effort="100" lower="-0.1" upper="1.1" velocity="1.0"/>
 		<calibration rising="0.0"/>
+		<origin xyz="0. -0.036 0.076" rpy="-1.57 0 0"/>
+		<axis xyz="0 0 0" />
 		</joint>
 	</robot>

Commit message: yaskawa gripper update

File: automatica2014_description/urdf/gripper.urdf.xacro (robot description, xacro)
@@ -4,5 +4,5 @@
     </xacro:property>
     <xacro:property name="flange_origin">
-        <origin xyz="0. 0. 0.03" rpy="0. 0 0" />
+        <origin xyz="0. 0. 0.03" rpy="0.0 0 1.5708" />
     </xacro:property>
      <link name="finger_left_link">

File: automatica2014_description/urdf/sia10f.urdf.xacro (robot description, xacro)
@@ -23,4 +23,5 @@
 		    <child link="gripper_grasp_link" />
 		    <xacro:insert_block name="gripper_origin" />
+		    <origin xyz="0.0 0.0 0.0" rpy="0 0 1.57"/>
 		</joint>
 		<joint name="finger_left_joint" type="prismatic" >
@@ -29,15 +30,14 @@
 		    <limit effort="100" lower="-0.01" upper="0.062" velocity="1.0"/>
 		    <calibration rising="0.0"/>
-		    <origin xyz="0.0 0.034 0.083" rpy="1.57 0 0"/>
+		    <origin xyz="0.0 0.0 0.096" rpy="-1.57 -1.57 3.14"/>
 		    <axis xyz="0 0 1" />
 		</joint>
 		<joint name="finger_right_joint" type="prismatic" >
-		<mimic joint="finger_left_joint" multiplier="-1" offset="0"/>
-		    <parent link="gripper_grasp_link" />
-		    <child link="finger_right_link" />
-		<limit effort="100" lower="-0.034" upper="0.01" velocity="1.0"/>
-		<calibration rising="0.0"/>
-		<origin xyz="0. -0.034 0.083" rpy="1.57 0 0"/>
-		<axis xyz="0 0 1" />
+			<parent link="gripper_grasp_link" />
+			<child link="finger_right_link" />
+			<limit effort="100" lower="-0.01" upper="0.062" velocity="1.0"/>
+			<calibration rising="0.0"/>
+			<origin xyz="0.0 0.0 0.096" rpy="-1.57 -1.57 0"/>
+			<axis xyz="0 0 1" />
 		</joint>
 	</robot>

Commit message: restructured gripper /sia10f URDF

File: automatica2014_description/urdf/gripper.urdf.xacro (robot description, xacro)
@@ -1,9 +1,3 @@
 <robot xmlns:xacro="http://ros.org/wiki/xacro">
-     <xacro:property name="gripper_origin">
-        <origin xyz="0. 0. 0" rpy="0 0 0" />
-    </xacro:property>
-    <xacro:property name="flange_origin">
-        <origin xyz="0. 0. 0.03" rpy="0.0 0 1.5708" />
-    </xacro:property>
      <link name="finger_left_link">
         <visual>
@@ -12,6 +6,6 @@
             </geometry>
             <material name="silver">
-					<color rgba="1 1 1 1"/>
-			</material>
+                            <color rgba="1 1 1 1"/>
+            </material>
         </visual>
         <collision>
@@ -20,6 +14,6 @@
             </geometry>
             <material name="silver">
-					<color rgba="1 1 1 1"/>
-			</material>
+                            <color rgba="1 1 1 1"/>
+            </material>
         </collision>
     </link>
@@ -30,6 +24,6 @@
             </geometry>
             <material name="silver">
-					<color rgba="1 1 1 1"/>
-			</material>
+                            <color rgba="1 1 1 1"/>
+            </material>
         </visual>
         <collision>
@@ -38,9 +32,9 @@
             </geometry>
             <material name="silver">
-					<color rgba="1 1 1 1"/>
-			</material>
+                            <color rgba="1 1 1 1"/>
+            </material>
         </collision>
     </link>
-    <link name="gripper_grasp_link">
+    <link name="gripper_link">
         <visual>
             <geometry>
@@ -48,6 +42,6 @@
             </geometry>
             <material name="blue">
-					<color rgba="0 0 1 1"/>
-			</material>
+                            <color rgba="0 0 1 1"/>
+            </material>
         </visual>
         <collision>
@@ -56,19 +50,23 @@
             </geometry>
             <material name="blue">
-					<color rgba="0 0 1 1"/>
-			</material>
+                            <color rgba="0 0 1 1"/>
+            </material>
         </collision>
     </link>
-    <link name="gripper_flange_link">
-        <visual>
-            <geometry>
-            <mesh filename="package://automatica2014_description/meshes/flange.stl"/>
-            </geometry>
-        </visual>
-        <collision>
-            <geometry>
-                <mesh filename="package://automatica2014_description/meshes/flange.stl"/>
-            </geometry>
-        </collision>
-    </link>
+    <joint name="finger_left_joint" type="prismatic" >
+        <parent link="gripper_link" />
+        <child link="finger_left_link" />
+        <limit effort="100" lower="-0.01" upper="0.062" velocity="1.0"/>
+        <calibration rising="0.0"/>
+        <origin xyz="0.0 0.0 0.096" rpy="-1.57 -1.57 3.14"/>
+        <axis xyz="0 0 1" />
+    </joint>
+    <joint name="finger_right_joint" type="prismatic" >
+            <parent link="gripper_link" />
+            <child link="finger_right_link" />
+            <limit effort="100" lower="-0.01" upper="0.062" velocity="1.0"/>
+            <calibration rising="0.0"/>
+            <origin xyz="0.0 0.0 0.096" rpy="-1.57 -1.57 0"/>
+            <axis xyz="0 0 1" />
+    </joint>
 </robot>

File: automatica2014_description/urdf/sia10f.urdf.xacro (robot description, xacro)
@@ -1,43 +1,50 @@
     <robot xmlns:xacro="http://ros.org/wiki/xacro" name="sia10f">
-		<xacro:include filename="$(find motoman_sia10f_support)/urdf/sia10f_macro.xacro" />
-		<!-- cell -->
-		<xacro:include filename="$(find automatica2014_description)/urdf/cell.urdf.xacro" />
-		 <!-- gripper and flange -->
-		<xacro:include filename="$(find automatica2014_description)/urdf/gripper.urdf.xacro" />
-		<!-- arm -->
-		<joint name="sia10f_base_joint" type="fixed" >
-		    <parent link="base_link" />
-		    <child link="sia10f_base_link" />
-		    <xacro:insert_block name="sia10f_origin" />
-		</joint>
-		<xacro:motoman_sia10f prefix="sia10f_"/>
-		<!-- gripper -->
-		<!-- gripper -->
-		<joint name="flange_joint" type="fixed" >
-		    <parent link="sia10f_link_t" />
-		    <child link="gripper_flange_link" />
-		    <xacro:insert_block name="flange_origin" />
-		</joint>
-		<joint name="gripper_joint" type="fixed" >
-		    <parent link="gripper_flange_link" />
-		    <child link="gripper_grasp_link" />
-		    <xacro:insert_block name="gripper_origin" />
-		    <origin xyz="0.0 0.0 0.0" rpy="0 0 1.57"/>
-		</joint>
-		<joint name="finger_left_joint" type="prismatic" >
-		    <parent link="gripper_grasp_link" />
-		    <child link="finger_left_link" />
-		    <limit effort="100" lower="-0.01" upper="0.062" velocity="1.0"/>
-		    <calibration rising="0.0"/>
-		    <origin xyz="0.0 0.0 0.096" rpy="-1.57 -1.57 3.14"/>
-		    <axis xyz="0 0 1" />
-		</joint>
-		<joint name="finger_right_joint" type="prismatic" >
-			<parent link="gripper_grasp_link" />
-			<child link="finger_right_link" />
-			<limit effort="100" lower="-0.01" upper="0.062" velocity="1.0"/>
-			<calibration rising="0.0"/>
-			<origin xyz="0.0 0.0 0.096" rpy="-1.57 -1.57 0"/>
-			<axis xyz="0 0 1" />
-		</joint>
-	</robot>
+                <xacro:property name="gripper_origin">
+                    <origin xyz="0. 0. 0" rpy="0 0 0" />
+                </xacro:property>
+                <xacro:property name="flange_origin">
+                    <origin xyz="0. 0. 0.03" rpy="0.0 0 1.5708" />
+                </xacro:property>
+                <xacro:include filename="$(find motoman_sia10f_support)/urdf/sia10f_macro.xacro" />
+                <!-- cell -->
+                <xacro:include filename="$(find automatica2014_description)/urdf/cell.urdf.xacro" />
+                 <!-- gripper and flange -->
+                <xacro:include filename="$(find automatica2014_description)/urdf/gripper.urdf.xacro" />
+                <!-- arm -->
+                <joint name="sia10f_base_joint" type="fixed" >
+                    <parent link="base_link" />
+                    <child link="sia10f_base_link" />
+                    <xacro:insert_block name="sia10f_origin" />
+                </joint>
+                <xacro:motoman_sia10f prefix="sia10f_"/>
+                <!-- gripper -->
+                <!-- gripper -->
+                <joint name="flange_joint" type="fixed" >
+                    <parent link="sia10f_link_t" />
+                    <child link="gripper_flange_link" />
+                    <xacro:insert_block name="flange_origin" />
+                </joint>
+                <link name="gripper_flange_link">
+                    <visual>
+                        <geometry>
+                        <mesh filename="package://automatica2014_description/meshes/flange.stl"/>
+                        </geometry>
+                    </visual>
+                    <collision>
+                        <geometry>
+                            <mesh filename="package://automatica2014_description/meshes/flange.stl"/>
+                        </geometry>
+                    </collision>
+                </link>
+                <joint name="gripper_joint" type="fixed" >
+                    <parent link="gripper_flange_link" />
+                    <child link="gripper_link" />
+                    <xacro:insert_block name="gripper_origin" />
+                </joint>
+                <joint name="gripper_grasp_joint" type="fixed" >
+                    <parent link="gripper_link" />
+                    <child link="gripper_grasp_link" />
+                    <origin xyz="0.0 0.0 0.0" rpy="0 0 0"/>
+                </joint>
+                <link name="gripper_grasp_link" />
+        </robot>

Commit message: Adds first ugly gripper model for ur5

File: automatica2014_description/urdf/gripper.urdf.xacro (robot description, xacro)
@@ -14,5 +14,5 @@
             </geometry>
             <material name="silver">
-                            <color rgba="1 1 1 1"/>
+                <color rgba="1 1 1 1"/>
             </material>
         </collision>
@@ -24,5 +24,5 @@
             </geometry>
             <material name="silver">
-                            <color rgba="1 1 1 1"/>
+                <color rgba="1 1 1 1"/>
             </material>
         </visual>
@@ -32,5 +32,5 @@
             </geometry>
             <material name="silver">
-                            <color rgba="1 1 1 1"/>
+                <color rgba="1 1 1 1"/>
             </material>
         </collision>
@@ -42,5 +42,5 @@
             </geometry>
             <material name="blue">
-                            <color rgba="0 0 1 1"/>
+                <color rgba="0 0 1 1"/>
             </material>
         </visual>
@@ -50,5 +50,5 @@
             </geometry>
             <material name="blue">
-                            <color rgba="0 0 1 1"/>
+                <color rgba="0 0 1 1"/>
             </material>
         </collision>

File: automatica2014_description/urdf/ur5.urdf.xacro (robot description, xacro)
@@ -14,5 +14,69 @@
         <parent link="ur5_wrist_3_link" />
         <child link="gripper_grasp_link" />
+        <origin xyz="0.0 0.06 0.0" rpy="1.57 0 0"/>
     </joint>
-    <link name="gripper_grasp_link" />
+    <link name="gripper_grasp_link">
+        <visual>
+            <geometry>
+                <mesh filename="package://automatica2014_description/meshes/gripper_base_lacquey.stl"/>
+            </geometry>
+        </visual>
+        <collision>
+            <geometry>
+                <mesh filename="package://automatica2014_description/meshes/gripper_base_lacquey.stl"/>
+            </geometry>
+        </collision>
+    </link>
+     <joint name="finger_left_joint" type="continuous" >
+        <parent link="gripper_grasp_link" />
+        <child link="finger_left_link" />
+        <limit effort="100" lower="-0.01" upper="0.062" velocity="1.0"/>
+        <calibration rising="0.0"/>
+        <origin xyz="-0.03 -0.03 -0.07" rpy="-1.57 0 0"/>
+        <axis xyz="0 0 1" />
+    </joint>
+    <link name="finger_left_link">
+        <visual>
+            <geometry>
+                <mesh filename="package://automatica2014_description/meshes/finger_right_lacquey.stl"/>
+            </geometry>
+            <material name="blue">
+                <color rgba="0 0 1 1"/>
+            </material>
+        </visual>
+        <collision>
+            <geometry>
+                <mesh filename="package://automatica2014_description/meshes/finger_right_lacquey.stl"/>
+            </geometry>
+            <material name="blue">
+                <color rgba="0 0 1 1"/>
+            </material>
+        </collision>
+    </link>
+     <joint name="finger_right_joint" type="continuous" >
+        <parent link="gripper_grasp_link" />
+        <child link="finger_right_link" />
+        <limit effort="100" lower="-0.01" upper="0.062" velocity="1.0"/>
+        <calibration rising="0.0"/>
+        <origin xyz="0.0 0.03 -0.07" rpy="-1.57 0 3.14"/>
+        <axis xyz="0 0 1" />
+    </joint>
+    <link name="finger_right_link">
+        <visual>
+            <geometry>
+                <mesh filename="package://automatica2014_description/meshes/finger_left_lacquey.stl"/>
+            </geometry>
+            <material name="blue">
+                <color rgba="0 0 1 1"/>
+            </material>
+        </visual>
+        <collision>
+            <geometry>
+                <mesh filename="package://automatica2014_description/meshes/finger_left_lacquey.stl"/>
+            </geometry>
+                <material name="blue">
+                <color rgba="0 0 1 1"/>
+            </material>
+        </collision>
+    </link>
 </robot>

Commit message: fix sia gripper

File: automatica2014_description/urdf/gripper.urdf.xacro (robot description, xacro)
@@ -59,5 +59,5 @@
         <limit effort="100" lower="-0.01" upper="0.062" velocity="1.0"/>
         <calibration rising="0.0"/>
-        <origin xyz="0.0 0.0 0.096" rpy="-1.57 -1.57 3.14"/>
+        <origin xyz="0.0 -0.008 0.096" rpy="-1.57 -1.57 3.14"/>
         <axis xyz="0 0 1" />
     </joint>
@@ -67,5 +67,5 @@
             <limit effort="100" lower="-0.01" upper="0.062" velocity="1.0"/>
             <calibration rising="0.0"/>
-            <origin xyz="0.0 0.0 0.096" rpy="-1.57 -1.57 0"/>
+            <origin xyz="0.0 0.008 0.096" rpy="-1.57 -1.57 0"/>
             <axis xyz="0 0 1" />
     </joint>

File: automatica2014_description/urdf/ur5.urdf.xacro (robot description, xacro)
@@ -83,5 +83,5 @@
         <parent link="gripper_link" />
         <child link="gripper_grasp_link" />
-        <origin xyz="0.0 0.06 0.0" rpy="1.57 0 0"/>
+        <origin xyz="0.0 0.06 0.0" rpy="3.14 0 -1.5708"/>
     </joint>
     <link name="gripper_grasp_link"/>

Commit message: moved Schunk STLs

File: automatica2014_description/urdf/gripper.urdf.xacro (robot description, xacro)
@@ -3,5 +3,5 @@
         <visual>
             <geometry>
-            <mesh filename="package://automatica2014_description/meshes/finger_left.stl"/>
+            <mesh filename="package://automatica2014_description/meshes/Schunk/finger_left_schunk.stl"/>
             </geometry>
             <material name="silver">
@@ -11,5 +11,5 @@
         <collision>
             <geometry>
-                <mesh filename="package://automatica2014_description/meshes/finger_left.stl"/>
+                <mesh filename="package://automatica2014_description/meshes/Schunk/finger_left_schunk.stl"/>
             </geometry>
             <material name="silver">
@@ -21,5 +21,5 @@
         <visual>
             <geometry>
-            <mesh filename="package://automatica2014_description/meshes/finger_right.stl"/>
+            <mesh filename="package://automatica2014_description/meshes/Schunk/finger_right_schunk.stl"/>
             </geometry>
             <material name="silver">
@@ -29,5 +29,5 @@
         <collision>
             <geometry>
-                <mesh filename="package://automatica2014_description/meshes/finger_right.stl"/>
+                <mesh filename="package://automatica2014_description/meshes/Schunk/finger_right_schunk.stl"/>
             </geometry>
             <material name="silver">
@@ -39,5 +39,5 @@
         <visual>
             <geometry>
-            <mesh filename="package://automatica2014_description/meshes/gripper.stl" scale="0.001 0.001 0.001"/>
+            <mesh filename="package://automatica2014_description/meshes/Schunk/gripper_schunk.stl" scale="0.001 0.001 0.001"/>
             </geometry>
             <material name="blue">
@@ -47,5 +47,5 @@
         <collision>
             <geometry>
-                <mesh filename="package://automatica2014_description/meshes/gripper.stl" scale="0.001 0.001 0.001"/>
+                <mesh filename="package://automatica2014_description/meshes/Schunk/gripper_schunk.stl" scale="0.001 0.001 0.001"/>
             </geometry>
             <material name="blue">
