Commit message: add launch and config for pg70

File: automatica2014_description/urdf/sia10f.urdf.xacro (robot description, xacro)
@@ -1,2 +1,3 @@
+<?xml version="1.0"?>
 <robot xmlns:xacro="http://ros.org/wiki/xacro" name="sia10f">
     <xacro:include filename="$(find motoman_sia10f_support)/urdf/sia10f_macro.xacro" />
@@ -15,4 +16,6 @@
         <parent link="sia10f_link_t" />
         <child link="gripper_grasp_link" />
+	<limit effort="100" lower="-0.1" upper="1.1" velocity="1.0"/>
+	<calibration rising="0.0"/>
     </joint>
     <link name="gripper_grasp_link" />

Commit message: First version of the gripper urdf

File: automatica2014_description/urdf/sia10f.urdf.xacro (robot description, xacro)
@@ -3,4 +3,6 @@
     <!-- cell -->
     <xacro:include filename="$(find automatica2014_description)/urdf/cell.urdf.xacro" />
+     <!-- gripper and flange -->
+    <xacro:include filename="$(find automatica2014_description)/urdf/gripper.urdf.xacro" />
     <!-- arm -->
     <joint name="sia10f_base_joint" type="fixed" >
@@ -12,8 +14,13 @@
     <!-- gripper -->
     <!-- gripper -->
+    <joint name="flange_joint" type="fixed" >
+        <parent link="sia10f_link_t" />
+        <child link="gripper_flange_link" />
+        <xacro:insert_block name="flange_origin" />
+    </joint>
     <joint name="gripper_joint" type="fixed" >
-        <parent link="sia10f_link_t" />
+        <parent link="gripper_flange_link" />
         <child link="gripper_grasp_link" />
+        <xacro:insert_block name="gripper_origin" />
     </joint>
-    <link name="gripper_grasp_link" />
 </robot>

Commit message: Some fixes for launching the gripper controller

File: automatica2014_description/urdf/sia10f.urdf.xacro (robot description, xacro)
@@ -22,4 +22,6 @@
 		    <parent link="gripper_flange_link" />
 		    <child link="gripper_grasp_link" />
+		    <limit effort="100" lower="-0.1" upper="1.1" velocity="1.0"/>
+		    <calibration rising="0.0"/>
 		    <xacro:insert_block name="gripper_origin" />
 		</joint>

Commit message: Added mimic joint for the fingers

File: automatica2014_description/urdf/sia10f.urdf.xacro (robot description, xacro)
@@ -24,18 +24,19 @@
 		    <xacro:insert_block name="gripper_origin" />
 		</joint>
-		<joint name="finger_left_joint" type="fixed" >
+		<joint name="finger_left_joint" type="revolute" >
 		    <parent link="gripper_grasp_link" />
 		    <child link="finger_left_link" />
 		    <limit effort="100" lower="-0.1" upper="1.1" velocity="1.0"/>
 		    <calibration rising="0.0"/>
-		    <origin xyz="0.0 0.044 0.076" rpy="-1.57 0 0"/>
+		    <origin xyz="0.0 0.034 0.083" rpy="1.57 0 0"/>
 		    <axis xyz="0 0 0" />
 		</joint>
-		<joint name="finger_right_joint" type="fixed" >
+		<joint name="finger_right_joint" type="revolute" >
+		<mimic joint="finger_left_joint" multiplier="1" offset="0"/>
 		    <parent link="gripper_grasp_link" />
 		    <child link="finger_right_link" />
 		<limit effort="100" lower="-0.1" upper="1.1" velocity="1.0"/>
 		<calibration rising="0.0"/>
-		<origin xyz="0. -0.036 0.076" rpy="-1.57 0 0"/>
+		<origin xyz="0. -0.034 0.083" rpy="1.57 0 0"/>
 		<axis xyz="0 0 0" />
 		</joint>

Commit message: removes unecessary limits from the gripper

File: automatica2014_description/urdf/sia10f.urdf.xacro (robot description, xacro)
@@ -22,6 +22,4 @@
 		    <parent link="gripper_flange_link" />
 		    <child link="gripper_grasp_link" />
-		    <limit effort="100" lower="-0.1" upper="1.1" velocity="1.0"/>
-		    <calibration rising="0.0"/>
 		    <xacro:insert_block name="gripper_origin" />
 		</joint>

Commit message: Fixes mimic joint urdf generation

File: automatica2014_description/urdf/sia10f.urdf.xacro (robot description, xacro)
@@ -24,5 +24,5 @@
 		    <xacro:insert_block name="gripper_origin" />
 		</joint>
-		<joint name="finger_left_joint" type="revolute" >
+		<joint name="finger_left_joint" type="prismatic" >
 		    <parent link="gripper_grasp_link" />
 		    <child link="finger_left_link" />
@@ -30,8 +30,8 @@
 		    <calibration rising="0.0"/>
 		    <origin xyz="0.0 0.034 0.083" rpy="1.57 0 0"/>
-		    <axis xyz="0 0 0" />
+		    <axis xyz="0 0 1" />
 		</joint>
-		<joint name="finger_right_joint" type="revolute" >
-		<mimic joint="finger_left_joint" multiplier="1" offset="0"/>
+		<joint name="finger_right_joint" type="prismatic" >
+		<mimic joint="finger_left_joint" multiplier="-1" offset="0"/>
 		    <parent link="gripper_grasp_link" />
 		    <child link="finger_right_link" />
@@ -39,5 +39,5 @@
 		<calibration rising="0.0"/>
 		<origin xyz="0. -0.034 0.083" rpy="1.57 0 0"/>
-		<axis xyz="0 0 0" />
+		<axis xyz="0 0 1" />
 		</joint>
 	</robot>

Commit message: Changes on the limits of the gripper

File: automatica2014_description/urdf/sia10f.urdf.xacro (robot description, xacro)
@@ -27,5 +27,5 @@
 		    <parent link="gripper_grasp_link" />
 		    <child link="finger_left_link" />
-		    <limit effort="100" lower="-0.1" upper="1.1" velocity="1.0"/>
+		    <limit effort="100" lower="-0.01" upper="0.062" velocity="1.0"/>
 		    <calibration rising="0.0"/>
 		    <origin xyz="0.0 0.034 0.083" rpy="1.57 0 0"/>
@@ -36,5 +36,5 @@
 		    <parent link="gripper_grasp_link" />
 		    <child link="finger_right_link" />
-		<limit effort="100" lower="-0.1" upper="1.1" velocity="1.0"/>
+		<limit effort="100" lower="-0.034" upper="0.01" velocity="1.0"/>
 		<calibration rising="0.0"/>
 		<origin xyz="0. -0.034 0.083" rpy="1.57 0 0"/>

Commit message: last night hacks

File: automatica2014_description/urdf/sia10f.urdf.xacro (robot description, xacro)
@@ -21,5 +21,5 @@
                 <!-- gripper -->
                 <joint name="flange_joint" type="fixed" >
-                    <parent link="sia10f_link_t" />
+                    <parent link="sia10f_link_7_t" />
                     <child link="gripper_flange_link" />
                     <xacro:insert_block name="flange_origin" />

Commit message: add collision for gripper grasp link

File: automatica2014_description/urdf/sia10f.urdf.xacro (robot description, xacro)
@@ -47,4 +47,11 @@
                     <origin xyz="0.0 0.0 0.14" rpy="0 3.14 1.5708"/>
                 </joint>
-                <link name="gripper_grasp_link" />
+                <link name="gripper_grasp_link" >
+                    <collision>
+                        <origin xyz="0.0 0.0 0.1" rpy="0 0 0"/>
+                        <geometry>
+                            <box size="0.01 0.01 0.01"/>
+                        </geometry>
+                    </collision>
+                </link>
         </robot>

Commit message: updated PGplus70 URDF

File: automatica2014_description/urdf/sia10f.urdf.xacro (robot description, xacro)
@@ -1,57 +1,48 @@
-    <robot xmlns:xacro="http://ros.org/wiki/xacro" name="sia10f">
-                <xacro:property name="gripper_origin">
-                    <origin xyz="0. 0. 0.0225" rpy="0 0 0" />
-                </xacro:property>
-                <xacro:property name="flange_origin">
-                    <origin xyz="0. 0. 0.03" rpy="0.0 0 1.5708" />
-                </xacro:property>
-                <xacro:include filename="$(find motoman_sia10f_support)/urdf/sia10f_macro.xacro" />
-                <!-- cell -->
-                <xacro:include filename="$(find automatica2014_description)/urdf/cell.urdf.xacro" />
-                 <!-- gripper and flange -->
-                <xacro:include filename="$(find automatica2014_description)/urdf/gripper.urdf.xacro" />
-                <!-- arm -->
-                <joint name="sia10f_base_joint" type="fixed" >
-                    <parent link="base_link" />
-                    <child link="sia10f_base_link" />
-                    <xacro:insert_block name="sia10f_origin" />
-                </joint>
-                <xacro:motoman_sia10f prefix="sia10f_"/>
-                <!-- gripper -->
-                <!-- gripper -->
-                <joint name="flange_joint" type="fixed" >
-                    <parent link="sia10f_link_7_t" />
-                    <child link="gripper_flange_link" />
-                    <xacro:insert_block name="flange_origin" />
-                </joint>
-                <link name="gripper_flange_link">
-                    <visual>
-                        <geometry>
-                        <mesh filename="package://automatica2014_description/meshes/flange.stl"/>
-                        </geometry>
-                    </visual>
-                    <collision>
-                        <geometry>
-                            <mesh filename="package://automatica2014_description/meshes/flange.stl"/>
-                        </geometry>
-                    </collision>
-                </link>
-                <joint name="gripper_joint" type="fixed" >
-                    <parent link="gripper_flange_link" />
-                    <child link="gripper_link" />
-                    <xacro:insert_block name="gripper_origin" />
-                </joint>
-                <joint name="gripper_grasp_joint" type="fixed" >
-                    <parent link="gripper_link" />
-                    <child link="gripper_grasp_link" />
-                    <origin xyz="0.0 0.0 0.14" rpy="0 3.14 1.5708"/>
-                </joint>
-                <link name="gripper_grasp_link" >
-                    <collision>
-                        <origin xyz="0.0 0.0 0.1" rpy="0 0 0"/>
-                        <geometry>
-                            <box size="0.01 0.01 0.01"/>
-                        </geometry>
-                    </collision>
-                </link>
-        </robot>
+<robot xmlns:xacro="http://ros.org/wiki/xacro" name="sia10f">
+    <xacro:include filename="$(find motoman_sia10f_support)/urdf/sia10f_macro.xacro" />
+    <xacro:include filename="$(find automatica2014_description)/urdf/PGplus70.urdf.xacro" />
+    <!-- cell -->
+    <xacro:include filename="$(find automatica2014_description)/urdf/cell.urdf.xacro" />
+    <!-- arm -->
+    <joint name="sia10f_base_joint" type="fixed" >
+        <parent link="base_link" />
+        <child link="sia10f_base_link" />
+        <xacro:insert_block name="sia10f_origin" />
+    </joint>
+    <xacro:motoman_sia10f prefix="sia10f_"/>
+    <!-- flange -->
+    <joint name="flange_joint" type="fixed" >
+        <parent link="sia10f_link_t" />
+        <child link="gripper_flange_link" />
+        <origin xyz="0. 0. 0.0" rpy="0.0 0 0" />
+    </joint>
+    <link name="gripper_flange_link">
+        <visual>
+            <origin xyz="0.0 0.0 0.025" rpy="0 0 0"/>   <!-- TODO -->
+            <geometry>
+                <cylinder radius="0.045" length="0.05"/>  <!-- TODO -->
+            </geometry>
+            <material name="white">
+                <color rgba="1 1 1 1"/>
+            </material>
+        </visual>
+    </link>
+    <!-- gripper -->
+    <xacro:PGplus70 prefix="" parent="gripper_flange_link">  <!-- TODO -->
+        <origin xyz="0.0 0.0 0.0525" rpy="0 0 1.57"/>
+    </xacro:PGplus70>
+    <!-- grasp point -->
+    <joint name="gripper_grasp_joint" type="fixed" >
+        <parent link="gripper_link" />
+        <child link="gripper_grasp_link" />
+        <origin xyz="0.0 0.0 0.14" rpy="0 3.14 1.5708"/>
+    </joint>
+    <link name="gripper_grasp_link" >
+        <collision>
+            <origin xyz="0.0 0.0 0.1" rpy="0 0 0"/>
+            <geometry>
+                <box size="0.01 0.01 0.01"/>
+            </geometry>
+        </collision>
+    </link>
+</robot>
