Commit message: clean-up

File: automatica2014_description/urdf/lacquey.urdf.xacro (robot description, xacro)
@@ -10,10 +10,10 @@
             <visual>
                 <geometry>
-                    <mesh filename="package://automatica2014_description/meshes/Lacquey/${prefix}gripper_base_lacquey.stl"/>
+                    <mesh filename="package://automatica2014_description/meshes/Lacquey/gripper_base_lacquey.stl"/>
                 </geometry>
             </visual>
             <collision>
                 <geometry>
-                    <mesh filename="package://automatica2014_description/meshes/Lacquey/${prefix}gripper_base_lacquey_coll.stl"/>
+                    <mesh filename="package://automatica2014_description/meshes/Lacquey/gripper_base_lacquey_coll.stl"/>
                 </geometry>
             </collision>

File: automatica2014_description/urdf/ur5.urdf.xacro (robot description, xacro)
@@ -11,8 +11,9 @@
     </joint>
     <xacro:ur5_robot prefix="ur5_"/>
+    <!-- gripper -->
     <xacro:lacquey_gripper prefix="" parent="ur5_ee_link">
         <origin xyz="0.0 0.0 0.0" rpy="0 1.57 0"/>
     </xacro:lacquey_gripper>
-    <!-- gripper -->
+    <!-- grasp link -->
     <joint name="gripper_grasp_joint" type="fixed" >
         <parent link="gripper_link" />

Commit message: updated Lacquey meshes

File: automatica2014_description/urdf/lacquey.urdf.xacro (robot description, xacro)
@@ -10,6 +10,7 @@
             <visual>
                 <geometry>
-                    <mesh filename="package://automatica2014_description/meshes/Lacquey/gripper_base_lacquey.stl"/>
+                    <mesh filename="package://automatica2014_description/meshes/Lacquey/gripper_base_lacquey.dae"/>
                 </geometry>
+                <origin xyz="0.0 -0.0025 0.0" rpy="0 0 0"/>
             </visual>
             <collision>
@@ -24,5 +25,5 @@
             <limit effort="100" lower="0" upper="1" velocity="1.0"/>
             <calibration rising="0.0"/>
-            <origin xyz="0.027 -0.0025 0.091" rpy="1.57 0 3.14"/>
+            <origin xyz="0.027 0 0.091" rpy="1.57 0 3.14"/>
             <axis xyz="0 0 1" />
         </joint>
@@ -30,5 +31,5 @@
             <visual>
                 <geometry>
-                    <mesh filename="package://automatica2014_description/meshes/Lacquey/finger_left_lacquey.stl"/>
+                    <mesh filename="package://automatica2014_description/meshes/Lacquey/finger_left_lacquey.dae"/>
                 </geometry>
                 <material name="blue">
@@ -50,5 +51,5 @@
             <limit effort="100" lower="0" upper="1" velocity="1.0"/>
             <calibration rising="0.0"/>
-            <origin xyz="-0.027 -0.0025 0.091" rpy="-1.57 0 0"/>
+            <origin xyz="-0.027 0 0.091" rpy="-1.57 0 0"/>
             <axis xyz="0 0 -1" />
         </joint>
@@ -56,5 +57,5 @@
             <visual>
                 <geometry>
-                    <mesh filename="package://automatica2014_description/meshes/Lacquey/finger_right_lacquey.stl"/>
+                    <mesh filename="package://automatica2014_description/meshes/Lacquey/finger_right_lacquey.dae"/>
                 </geometry>
                 <material name="blue">
