Commit message: currect finger position

File: automatica2014_description/urdf/PGplus70.urdf.xacro (robot description, xacro)
@@ -29,5 +29,5 @@
                 <limit effort="100" lower="0.001" upper="0.0345" velocity="2.0"/>
                 <calibration rising="0.0"/>
-                <origin xyz="0 0.0105 0.08" rpy="0 0 1.5708"/>
+                <origin xyz="0 0.0105 0.0789" rpy="0 0 1.5708"/>
                 <axis xyz="1 0 0" />
         </joint>
@@ -55,5 +55,5 @@
                 <limit effort="100" lower="0.001" upper="0.0345" velocity="2.0"/>
                 <calibration rising="0.0"/>
-                <origin xyz="0 -0.0105 0.08" rpy="-0 0 -1.5708"/>
+                <origin xyz="0 -0.0105 0.0789" rpy="-0 0 -1.5708"/>
                 <axis xyz="1 0 0" />
         </joint>

Commit message: dae mesh for Schunk gripper

File: automatica2014_description/urdf/PGplus70.urdf.xacro (robot description, xacro)
@@ -9,5 +9,5 @@
                 <visual>
                     <geometry>
-                    <mesh filename="package://automatica2014_description/meshes/Schunk/gripper_schunk.stl" scale="0.001 0.001 0.001"/>
+                    <mesh filename="package://automatica2014_description/meshes/Schunk/gripper_schunk.dae" scale="0.001 0.001 0.001"/>
                     </geometry>
                     <material name="blue">

Commit message: use the DAE as collision model too

File: automatica2014_description/urdf/PGplus70.urdf.xacro (robot description, xacro)
@@ -17,5 +17,5 @@
                 <collision>
                     <geometry>
-                        <mesh filename="package://automatica2014_description/meshes/Schunk/gripper_schunk.stl" scale="0.001 0.001 0.001"/>
+                        <mesh filename="package://automatica2014_description/meshes/Schunk/gripper_schunk.dae" scale="0.001 0.001 0.001"/>
                     </geometry>
                     <material name="blue">
